File: bmb/typec-v1.0/bitmagic-basic.kicad_pcb (KiCad board)
At the start: 4 copper layers, 40 x 16 mm, 43 parts, among them IC1 CY7C68013A-56, J1 Conn_02x05_Odd_Even, J2 Host_USB_C, U1 3.3V, U2 USBLC6-2, U3 IP425x-4-TTL, U4 IP425x-4-TTL, U5 24LC00, U6 IP425x-4-TTL, X1 24MHz

Commit message: Renamed v1.0c to Type-C
Other:
- board text added: "BitMagic Type-C"
- board text added: "Type-C"
- board text added: "V1.0"
- board text added: "V1.0 CC-BY-SA 4.0"
- board text removed: "Basic"
- board text removed: "BitMagic Basic"
- board text removed: "V1.0c"
- board text removed: "V1.0c CC-BY-SA 4.0"
Changed lines of the file:
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@@
     (effects (font (size 1 1) (thickness 0.15)))
   )
-  (gr_text Basic (at 41.2 25) (layer F.SilkS)
+  (gr_text Type-C (at 41.2 25) (layer F.SilkS)
     (effects (font (size 1 1) (thickness 0.25)))
   )
-  (gr_text "V1.0c\nCC-BY-SA 4.0" (at 23.4 30 270) (layer B.SilkS)
+  (gr_text "V1.0\nCC-BY-SA 4.0" (at 23.4 30 270) (layer B.SilkS)
     (effects (font (size 1 1) (thickness 0.25)) (justify mirror))
   )
-  (gr_text "BitMagic Basic" (at 26.9 30 270) (layer B.SilkS)
-    (effects (font (size 1.3 1.3) (thickness 0.3)) (justify mirror))
+  (gr_text "BitMagic Type-C" (at 26.9 30 270) (layer B.SilkS)
+    (effects (font (size 1.2 1.2) (thickness 0.3)) (justify mirror))
   )
   (gr_line (start 38.5 21) (end 38.5 39) (layer Dwgs.User) (width 0.2))
-  (gr_text V1.0c (at 47.1 23.5) (layer F.SilkS)
+  (gr_text V1.0 (at 47.1 23.5) (layer F.SilkS)
     (effects (font (size 1 1) (thickness 0.25)))
   )

Commit message: Factory 0402 footprint to pkl 0402, silkscreen fixes
The USB Type C 5k1 resistors used factory KiCAD footprints and are now pkl as all the others.
Pin 6 is now correctly marked
Parts:
- R10, R11, R12: footprint Resistor_SMD:R_0402_1005Metric -> pkl_dipol:R_0402
Other:
- board text added: "6"
- board text removed: "8"
